Commit message: Uploaded ball_chaser

File: src/my_robot/urdf/my_robot.xacro (robot description, xacro)
@@ -71,5 +71,5 @@
       <origin xyz="0 0 0" rpy=" 0 1.5707 1.5707"/>
       <geometry>
-        <cylinder radius='.1' length='.05'/>
+        <cylinder radius='.101' length='.05'/>
       </geometry>
     </collision>
@@ -77,10 +77,10 @@
       <origin xyz="0 0 0" rpy=" 0 1.5707 1.5707"/>
       <geometry>
-        <cylinder radius='.1' length='.05'/>
+        <cylinder radius='.101' length='.05'/>
       </geometry>
     </visual>
   </link>
   <joint type="continuous" name="left_wheel_hinge">
-    <origin xyz="0 0.15 0" rpy="0 0 0"/>
+    <origin xyz="0 0.21 0" rpy="0 0 0"/>
     <child link="left_wheel"/>
     <parent link="chassis"/>
@@ -102,5 +102,5 @@
       <origin xyz="0 0 0" rpy=" 0 1.5707 1.5707"/>
       <geometry>
-        <cylinder radius='.1' length='.05'/>
+        <cylinder radius='.101' length='.05'/>
       </geometry>
     </collision>
@@ -108,10 +108,10 @@
       <origin xyz="0 0 0" rpy=" 0 1.5707 1.5707"/>
       <geometry>
-        <cylinder radius='.1' length='.05'/>
+        <cylinder radius='.101' length='.05'/>
       </geometry>
     </visual>
   </link>
   <joint type="continuous" name="right_wheel_hinge">
-    <origin xyz="0 -0.15 0" rpy="0 0 0"/>
+    <origin xyz="0 -0.21 0" rpy="0 0 0"/>
     <child link="right_wheel"/>
     <parent link="chassis"/>
